File: BP-PCB-Kicad.kicad_pcb (KiCad board)
At the start: 2 copper layers, 98 x 120.7 mm, 18 parts, among them J10 A3C-4DA-2DSA_71_, J12 A3C-4DA-2DSA_71_, J16 DF14-15P-1.25H52, J17 DF14-30P-1.25H_35_, J18 DF14-15P-1.25H52, J19 DF14-15P-1.25H52, J20 A3C-50DA-2DSA_71_, J21 A3C-50DA-2DSA_71_, J22 A3C-50DA-2DSA_71_, J23 A3C-50DA-2DSA_71_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

Commit message: Git Submodule added inside <KiCad-Libaries> folder to share libraries across different projects
Parts:
- J10, J12: footprint BPB-Footprints:Hirose_A3C-4DA-2DSA(71) -> Custom-Footprints:Hirose_A3C-4DA-2DSA(71)
- J16, J18, J19: footprint BPB-Footprints:Hirose_DF14-15P-1.25H(52) -> Custom-Footprints:Hirose_DF14-15P-1.25H(52)
- J17: footprint BPB-Footprints:Hirose_DF14-30P-1.25H(35) -> Custom-Footprints:Hirose_DF14-30P-1.25H(35)
- J20, J21, J23: footprint BPB-Footprints:Hirose_A3C-50DA-2DSC(71) -> Custom-Footprints:Hirose_A3C-50DA-2DSC(71)
- J22, J24: footprint BPB-Footprints:Hirose_A3C-50DA-2DSC(71)_Mirrored -> Custom-Footprints:Hirose_A3C-50DA-2DSC(71)_Mirrored
- J25, J26, J27: footprint BPB-Footprints:Molex_0554600272 -> Custom-Footprints:Molex_0554600272
- J28: footprint BPB-Footprints:PSR-210153-20_P2.00mm -> Custom-Footprints:PSR-210153-20_P2.00mm
- J29: footprint BPB-Footprints:PSR-210153-20_P2.00mm_Mirrored -> Custom-Footprints:PSR-210153-20_P2.00mm_Mirrored
- J7, J9: footprint BPB-Footprints:Hirose_A3C-4DA-2DSA(71)_Mirrored -> Custom-Footprints:Hirose_A3C-4DA-2DSA(71)_Mirrored
Changed lines of the file:
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@@
 	(net 201 "unconnected-(J19-PadMP1)")
 	(net 202 "unconnected-(J19-PadMP2)")
-	(footprint "BPB-Footprints:Molex_0554600272"
+	(footprint "Custom-Footprints:Molex_0554600272"
 		(layer "F.Cu")
 		(at 111.55 119.47 90)
@@
 		)
 		(embedded_fonts no)
-		(model "${KIPRJMOD}/3Ds/Molex_554600272.stp"
+		(model "${KIPRJMOD}/KiCad-Libraries/3Ds/Molex_554600272.stp"
 			(offset
 				(xyz -1 -2.24 3.4)
@@
 		)
 	)
-	(footprint "BPB-Footprints:Hirose_A3C-50DA-2DSC(71)_Mirrored"
+	(footprint "Custom-Footprints:Hirose_A3C-50DA-2DSC(71)_Mirrored"
 		(layer "F.Cu")
 		(at 45 22.52)
@@
 		)
 		(embedded_fonts no)
-		(model "/Users/akramov/Documents/Turan1/BPB/PCB-Component-Files/LIB_A3C-50DA-2DSA_71_/A3C-50DA-2DSA_71_/3D/A3C-50DA-2DSA.stp"
+		(model "${KIPRJMOD}/KiCad-Libraries/3Ds/Hirose A3C-50DA-2DSA(71).stp"
 			(offset
 				(xyz 24 -1 0)
@@
 		)
 	)
-	(footprint "BPB-Footprints:Molex_0554600272"
+	(footprint "Custom-Footprints:Molex_0554600272"
 		(layer "F.Cu")
 		(at 26.45 121.47 -90)
@@
 		)
 		(embedded_fonts no)
-		(model "${KIPRJMOD}/3Ds/Molex_554600272.stp"
+		(model "${KIPRJMOD}/KiCad-Libraries/3Ds/Molex_554600272.stp"
 			(offset
 				(xyz -1 -2.24 3.4)
@@
 		)
 	)
-	(footprint "BPB-Footprints:Hirose_A3C-4DA-2DSA(71)"
+	(footprint "Custom-Footprints:Hirose_A3C-4DA-2DSA(71)"
 		(layer "F.Cu")
 		(at 40 89.02)
@@
 		)
 		(embedded_fonts no)
-		(model "${KIPRJMOD}/3Ds/Hirose A3C-4DA-2DSA(71).step"
+		(model "${KIPRJMOD}/KiCad-Libraries/3Ds/Hirose A3C-4DA-2DSA(71).step"
 			(offset
 				(xyz 24 1 0)
@@
 		)
 	)
-	(footprint "BPB-Footprints:Hirose_A3C-50DA-2DSC(71)"
+	(footprint "Custom-Footprints:Hirose_A3C-50DA-2DSC(71)"
 		(layer "F.Cu")
 		(at 45 129)
@@
 		)
 		(embedded_fonts no)
-		(model "${KIPRJMOD}/3Ds/Hirose A3C-50DA-2DSA(71).stp"
+		(model "${KIPRJMOD}/KiCad-Libraries/3Ds/Hirose A3C-50DA-2DSA(71).stp"
 			(offset
 				(xyz 24 1 0)
@@
 		)
 	)
-	(footprint "BPB-Footprints:Hirose_A3C-50DA-2DSC(71)"
+	(footprint "Custom-Footprints:Hirose_A3C-50DA-2DSC(71)"
 		(layer "F.Cu")
 		(at 45 111.42)
@@
 		)
 		(embedded_fonts no)
-		(model "${KIPRJMOD}/3Ds/Hirose A3C-50DA-2DSA(71).stp"
+		(model "${KIPRJMOD}/KiCad-Libraries/3Ds/Hirose A3C-50DA-2DSA(71).stp"
 			(offset
 				(xyz 24 1 0)
@@
 		)
 	)
-	(footprint "BPB-Footprints:PSR-210153-20_P2.00mm"
+	(footprint "Custom-Footprints:PSR-210153-20_P2.00mm"
 		(layer "F.Cu")
 		(at 115 57.02)
@@
 		)
 		(embedded_fonts no)
-		(model "${KIPRJMOD}/3Ds/PSR-210153-20-Male.STEP"
+		(model "${KIPRJMOD}/KiCad-Libraries/3Ds/PSR-210153-20-Male.STEP"
 			(offset
 				(xyz 1 1.05 0)
@@
 		)
 	)
-	(footprint "BPB-Footprints:Hirose_A3C-4DA-2DSA(71)_Mirrored"
+	(footprint "Custom-Footprints:Hirose_A3C-4DA-2DSA(71)_Mirrored"
 		(layer "F.Cu")
 		(at 40 101.43)
@@
 		)
 		(embedded_fonts no)
-		(model "${KIPRJMOD}/3Ds/Hirose A3C-4DA-2DSA(71).step"
+		(model "${KIPRJMOD}/KiCad-Libraries/3Ds/Hirose A3C-4DA-2DSA(71).step"
 			(offset
 				(xyz 24 -1 0)
@@
 		)
 	)
-	(footprint "BPB-Footprints:Molex_0554600272"
+	(footprint "Custom-Footprints:Molex_0554600272"
 		(layer "F.Cu")
 		(at 111.55 105.48 90)
@@
 		)
 		(embedded_fonts no)
-		(model "${KIPRJMOD}/3Ds/Molex_554600272.stp"
+		(model "${KIPRJMOD}/KiCad-Libraries/3Ds/Molex_554600272.stp"
 			(offset
 				(xyz -1 -2.24 3.4)
@@
 		)
 	)
-	(footprint "BPB-Footprints:Hirose_A3C-50DA-2DSC(71)_Mirrored"
+	(footprint "Custom-Footprints:Hirose_A3C-50DA-2DSC(71)_Mirrored"
 		(layer "F.Cu")
 		(at 45 101.43)
@@
 		)
 		(embedded_fonts no)
-		(model "/Users/akramov/Documents/Turan1/BPB/PCB-Component-Files/LIB_A3C-50DA-2DSA_71_/A3C-50DA-2DSA_71_/3D/A3C-50DA-2DSA.stp"
+		(model "${KIPRJMOD}/KiCad-Libraries/3Ds/Hirose A3C-50DA-2DSA(71).stp"
 			(offset
 				(xyz 24 -1 0)
@@
 		)
 	)
-	(footprint "BPB-Footprints:Hirose_A3C-4DA-2DSA(71)_Mirrored"
+	(footprint "Custom-Footprints:Hirose_A3C-4DA-2DSA(71)_Mirrored"
 		(layer "F.Cu")
 		(at 96 101.43)
@@
 		)
 		(embedded_fonts no)
-		(model "${KIPRJMOD}/3Ds/Hirose A3C-4DA-2DSA(71).step"
+		(model "${KIPRJMOD}/KiCad-Libraries/3Ds/Hirose A3C-4DA-2DSA(71).step"
 			(offset
 				(xyz 24 -1 0)
@@
 		)
 	)
-	(footprint "BPB-Footprints:Hirose_A3C-50DA-2DSC(71)"
+	(footprint "Custom-Footprints:Hirose_A3C-50DA-2DSC(71)"
 		(layer "F.Cu")
 		(at 45 89.02)
@@
 		)
 		(embedded_fonts no)
-		(model "${KIPRJMOD}/3Ds/Hirose A3C-50DA-2DSA(71).stp"
+		(model "${KIPRJMOD}/KiCad-Libraries/3Ds/Hirose A3C-50DA-2DSA(71).stp"
 			(offset
 				(xyz 24 1 0)
@@
 		)
 	)
-	(footprint "BPB-Footprints:PSR-210153-20_P2.00mm_Mirrored"
+	(footprint "Custom-Footprints:PSR-210153-20_P2.00mm_Mirrored"
 		(layer "F.Cu")
 		(at 23 57.02)
@@
 		)
 		(embedded_fonts no)
-		(model "${KICAD9_3DMODEL_DIR}/Connector_PinHeader_2.00mm.3dshapes/PinHeader_1x20_P2.00mm_Horizontal.step"
-			(hide yes)
-			(offset
-				(xyz 0 -38 0)
-			)
-			(scale
-				(xyz 1 1 1)
-			)
-			(rotate
-				(xyz -0 -180 -0)
-			)
-		)
-		(model "${KIPRJMOD}/3Ds/PSR-210153-20-Male.STEP"
+		(model "${KIPRJMOD}/KiCad-Libraries/3Ds/PSR-210153-20-Male.STEP"
 			(offset
-				(xyz -1 -39 0)
+				(xyz -1 -39.05 0)
 			)
 			(scale
@@
 			)
 			(rotate
-				(xyz -180 180 90)
+				(xyz 180 -180 90)
 			)
 		)
 	)
-	(footprint "BPB-Footprints:Hirose_A3C-4DA-2DSA(71)"
+	(footprint "Custom-Footprints:Hirose_A3C-4DA-2DSA(71)"
 		(layer "F.Cu")
 		(at 96 89.02)
@@
 		)
 		(embedded_fonts no)
-		(model "${KIPRJMOD}/3Ds/Hirose A3C-4DA-2DSA(71).step"
+		(model "${KIPRJMOD}/KiCad-Libraries/3Ds/Hirose A3C-4DA-2DSA(71).step"
 			(offset
 				(xyz 24 1 0)
@@
 		)
 	)
-	(footprint "BPB-Footprints:Hirose_DF14-15P-1.25H(52)"
+	(footprint "Custom-Footprints:Hirose_DF14-15P-1.25H(52)"
 		(layer "B.Cu")
 		(at 99.9 77.5 180)
@@
 		)
 		(embedded_fonts no)
-		(model "/Users/akramov/Documents/Turan1/BPB/PCB-Component-Files/DF14-15P-1.25H(52)/DF14-15P-1.25H.stp"
+		(model "${KIPRJMOD}/KiCad-Libraries/3Ds/Hirose DF14-15P-1.25H.stp"
 			(offset
 				(xyz 21.15 2.25 0)
@@
 		)
 	)
-	(footprint "BPB-Footprints:Hirose_DF14-15P-1.25H(52)"
+	(footprint "Custom-Footprints:Hirose_DF14-15P-1.25H(52)"
 		(layer "B.Cu")
 		(at 46.1 114.5)
@@
 		)
 		(embedded_fonts no)
-		(model "/Users/akramov/Documents/Turan1/BPB/PCB-Component-Files/DF14-15P-1.25H(52)/DF14-15P-1.25H.stp"
+		(model "${KIPRJMOD}/KiCad-Libraries/3Ds/Hirose DF14-15P-1.25H.stp"
 			(offset
 				(xyz 21.15 2.25 0)
@@
 		)
 	)
-	(footprint "BPB-Footprints:Hirose_DF14-30P-1.25H(35)"
+	(footprint "Custom-Footprints:Hirose_DF14-30P-1.25H(35)"
 		(layer "B.Cu")
 		(at 74.35 77.5 180)
@@
 		)
 		(embedded_fonts no)
-		(model "${KIPRJMOD}/3Ds/Hirose DF14-30P-1.25H(35).STEP"
+		(model "${KIPRJMOD}/KiCad-Libraries/3Ds/Hirose DF14-30P-1.25H(35).STEP"
 			(offset
 				(xyz -15.95 2.3 -0.05)
@@
 		)
 	)
-	(footprint "BPB-Footprints:Hirose_DF14-15P-1.25H(52)"
+	(footprint "Custom-Footprints:Hirose_DF14-15P-1.25H(52)"
 		(layer "B.Cu")
 		(at 74.4 114.5)
@@
 		)
 		(embedded_fonts no)
-		(model "/Users/akramov/Documents/Turan1/BPB/PCB-Component-Files/DF14-15P-1.25H(52)/DF14-15P-1.25H.stp"
+		(model "${KIPRJMOD}/KiCad-Libraries/3Ds/Hirose DF14-15P-1.25H.stp"
 			(offset
 				(xyz 21.15 2.25 0)
