File: _autosave-BP-PCB-Kicad.kicad_pcb (KiCad board)
At the start: 4 copper layers, 120.7 x 98 mm, 74 parts, among them IC1 LMT84DCKT, J1 A3C-50DA-2DSA_71_, J13 Conn_01x20, J14 Conn_01x20, J15 DF14-30P-1.25H_35_, J16 A3C-50DA-2DSA_71_, J17 A3C-4DA-2DSA_71_, J18 A3C-4DA-2DSA_71_, J19 Molex 55460-0272, J2 A3C-50DA-2DSA_71_, J21 Molex 55460-0272, J22 Molex 55460-0272, J23 DF14-15P-1.25H52, J3 A3C-4DA-2DSA_71_, J4 A3C-4DA-2DSA_71_, J5 A3C-50DA-2DSA_71_, J6 A3C-50DA-2DSA_71_, J7 DF14-15P-1.25H52, J8 DF14-15P-1.25H52, Q1 SSM6K514NU,LF, Q2 SSM6K514NU,LF, Q3 SSM6K514NU,LF, Q4 SSM6K514NU,LF, Q5 SSM6K514NU,LF, Q6 SSM6K514NU,LF, U1 LTC4361CTS8-2TRMPBF, U2 LTC4361CTS8-2TRMPBF, U3 SN74CB3Q3257DBQR, U5 SN74CB3Q3257DBQR, U6 LTC4389IMS-4#PBF, U7 LTC4389IMS-4#PBF

Commit message: Finished routing v1
Routing:
- net  V_IN (Unreg2 OCP to S-band RX): track 136.6 -> 131.9 mm
Changed lines of the file:
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@@
 	)
 	(via
-		(at 58.12 121.51)
+		(at 58.12 118.15)
 		(size 0.6)
 		(drill 0.3)
@@
 	)
 	(segment
-		(start 56.293 95.2)
-		(end 54.81 96.683)
-		(width 0.3)
-		(layer "B.Cu")
-		(net 17)
-	)
-	(segment
-		(start 56.925 95.2)
-		(end 56.293 95.2)
-		(width 0.3)
-		(layer "B.Cu")
-		(net 17)
-	)
-	(segment
-		(start 54.81 96.683)
-		(end 54.81 118.2)
+		(start 58.11 118.15)
+		(end 54.81 114.85)
 		(width 0.3)
 		(layer "B.Cu")
@@
 	)
 	(segment
+		(start 54.81 96.683)
+		(end 56.293 95.2)
+		(width 0.3)
+		(layer "B.Cu")
+		(net 17)
+	)
+	(segment
+		(start 56.293 95.2)
+		(end 56.925 95.2)
+		(width 0.3)
+		(layer "B.Cu")
+		(net 17)
+	)
+	(segment
+		(start 58.12 118.15)
+		(end 58.11 118.15)
+		(width 0.3)
+		(layer "B.Cu")
+		(net 17)
+	)
+	(segment
 		(start 122 96.9925)
 		(end 122.01 97.0025)
 		(width 0.25)
+		(layer "B.Cu")
+		(net 17)
+	)
+	(segment
+		(start 54.81 114.85)
+		(end 54.81 96.683)
+		(width 0.3)
 		(layer "B.Cu")
 		(net 17)
@@
 	)
 	(segment
-		(start 54.81 118.2)
-		(end 58.12 121.51)
-		(width 0.3)
-		(layer "B.Cu")
-		(net 17)
-	)
-	(segment
 		(start 114.93 96.99)
 		(end 118.8075 96.99)
@@
 	)
 	(segment
-		(start 118.8 118.13)
+		(start 58.12 118.15)
+		(end 58.13 118.14)
+		(width 0.3)
+		(layer "In1.Cu")
+		(net 17)
+	)
+	(segment
+		(start 114.92 118.14)
 		(end 114.93 118.13)
 		(width 0.3)
@@
 	)
 	(segment
-		(start 114.93 118.13)
+		(start 58.13 118.14)
 		(end 114.92 118.14)
 		(width 0.3)
@@
 	)
 	(segment
-		(start 61.49 118.14)
-		(end 58.12 121.51)
+		(start 114.93 118.13)
+		(end 118.8 118.13)
 		(width 0.3)
 		(layer "In1.Cu")
-		(net 17)
-	)
-	(segment
-		(start 114.92 118.14)
-		(end 61.49 118.14)
-		(width 0.3)
-		(layer "In1.Cu")
