File: BP-PCB-Kicad.kicad_sch (KiCad schematic)
At the start: 23 parts, among them J1 Conn_02x25_Odd_Even, J10 A3C-4DA-2DSA_71_, J11 Conn_02x25_Odd_Even, J12 A3C-4DA-2DSA_71_, J15 Conn_02x25_Odd_Even, J16 DF14-15P-1.25H52, J17 DF14-30P-1.25H_35_, J18 DF14-15P-1.25H52, J19 DF14-15P-1.25H52, J20 A3C-50DA-2DSA_71_, J21 A3C-50DA-2DSA_71_, J22 A3C-50DA-2DSA_71_, J23 A3C-50DA-2DSA_71_, J24 A3C-50DA-2DSA_71_, J25 Molex 55460-0272, J26 Molex 55460-0272, J27 Molex 55460-0272, J28 Conn_01x20, J29 Conn_01x20, J5 Conn_02x25_Odd_Even, J7 A3C-4DA-2DSA_71_, J8 Conn_02x25_Odd_Even, J9 A3C-4DA-2DSA_71_

Commit message: Fixed errors in schematics
Parts:
- removed J1, J11, J15, J5, J8: Conn_02x25_Odd_Even, symbol Connector_Generic:Conn_02x25_Odd_Even
- renumbered J20 to J1, J21 to J10, J28 to J13, J29 to J14, J17 to J15, J22 to J16, J7 to J17, J9 to J18, J25 to J19, J23 to J2, J27 to J21, J26 to J22, J19 to J23, J10 to J3, J12 to J4, J16 to J7, J18 to J8, J24 to J9
Connections:
- net GND_SYS: now also J13.19 (Pin_19), J13.20 (Pin_20), J14.19 (Pin_19), J14.2 (Pin_2); no longer J13.17 (Pin_17), J13.18 (Pin_18), J14.13 (Pin_13), J14.14 (Pin_14)
- net GPS_1PPS: now also J13.16 (Pin_16); no longer J13.14 (Pin_14)
- net GPS_3v3: now also J13.15 (Pin_15); no longer J13.13 (Pin_13)
- net POWERSC_+X: now also J14.13 (Pin_13), J14.14 (Pin_14), J14.15 (Pin_15), J14.16 (Pin_16); no longer J14.4 (Pin_4), J14.5 (Pin_5), J14.6 (Pin_6), J14.7 (Pin_7)
- net POWERSC_+Y: now also J14.6 (Pin_6), J14.7 (Pin_7); no longer J14.17 (Pin_17), J14.18 (Pin_18)
- net POWERSC_-X1: now also J13.7 (Pin_7), J13.8 (Pin_8); no longer J13.4 (Pin_4), J13.5 (Pin_5)
- net POWERSC_-X2: now also J13.13 (Pin_13), J13.14 (Pin_14); no longer J13.7 (Pin_7), J13.8 (Pin_8)
- net Sunsensor_+X: now also J14.18 (Pin_18); no longer J14.8 (Pin_8)
- net Sunsensor_+Y: now also J14.10 (Pin_10); no longer J14.19 (Pin_19)
- net TEMP_+X: now also J14.17 (Pin_17); no longer J14.2 (Pin_2)
- net TEMP_+Y: now also J14.4 (Pin_4); no longer J14.16 (Pin_16)
- net TEMP_+Z: now also J14.11 (Pin_11); no longer J14.15 (Pin_15)
- net UART (ADCS_to_GPS): now also J13.18 (Pin_18); no longer J13.16 (Pin_16)
- net UART (GPS_to_ADCS): now also J13.17 (Pin_17); no longer J13.15 (Pin_15)
- net FSS-M1-ES_SCL: no longer names the net of J9.38
- net FSS-M1-ES_SCL: no longer J13.12 (Pin_12)
- net FSS-M1-ES_SDA: no longer names the net of J9.37
- net FSS-M1-ES_SDA: no longer J13.11 (Pin_11)
- net FSS-M1_3v3: no longer names the net of J9.33
- net FSS-M1_3v3: no longer J13.10 (Pin_10)
- net FSS-M2_3v3: no longer names the net of J9.34
- net FSS-M2_3v3: no longer J14.9 (Pin_9)
- net FSS-M2_SCL: no longer names the net of J9.40
- net FSS-M2_SCL: no longer J14.11 (Pin_11)
- net FSS-M2_SDA: no longer names the net of J9.39
- net FSS-M2_SDA: no longer J14.10 (Pin_10)
- no-connect marks 69 -> 81

Commit message: Synchronized with pin mapping table and added circuits
Parts:
- J13: footprint Custom-Footprints:PSR-210153-20_P2.00mm -> Custom-Footprints:PSR-420253-10
- J14: footprint Custom-Footprints:PSR-210153-20_P2.00mm_Mirrored -> Custom-Footprints:PSR-420253-10_Mirrored
Connections:
- net Sunsensor_-Z is gone; now on net Sunsensor_-Z1: J9.12
- net GND_SYS: now also J13.2 (Pin_2)
- net OBC-ADCS_DIO_ON/OFF (MainPIC_to_ADCS): now also J9.46; no longer J9.6
- net SUP_5V_1: no longer J1.16
- net SUP_5V_2: no longer J1.25, J1.26
- net SUP_UNREG_2: no longer J1.35, J1.36
- net TEMP_-X: now also J13.3 (Pin_3); no longer J13.2 (Pin_2)
- net TEMP_-Z: now also J14.5 (Pin_5)
- net Sunsensor_-Z2: now reaches J9.21
- net Sunsensor_-Z2: now also J14.9 (Pin_9)
- net E-MGM_3v3: now reaches J9.33
- net E-MGM_3v3: now also J13.10 (Pin_10)
- net E-MGM_SDA: now reaches J9.37
- net E-MGM_SDA: now also J13.11 (Pin_11)
- net E-MGM_SCL: now reaches J9.38
- net E-MGM_SCL: now also J13.12 (Pin_12)
- net Sunsensor_-Z1: now reaches J14.8 (Pin_8)
- net TEMP_3v3_MX: now reaches J13.4 (Pin_4)
- net DIO S-band RX ON/OFF renamed DIO_S-Band_RX_ON/OFF
- net OBC-SBAND_TX_ON/OFF renamed DIO_S-Band_TX_ON/OFF
- net TEMP_3v3 renamed TEMP_3v3_PX
- net TEMP_3v3_PX: no longer J13.3 (Pin_3)
- no-connect marks 81 -> 75
Other:
- sheet BP-PCB-ICs renamed BP-PCB-ICs-1
- added sheet BP_PCB-ICs-2 (BP_PCB-ICs-2.kicad_sch)

Commit message: PCB layout is syncronized with schematic
Connections:
- net OBC-CCB DIO ON/OFF (MainPIC_to_CCB) is gone; now on net OBC-CCB_DIO_ON/OFF (MainPIC_to_CCB): J15.1
- net POWERSC_-X_1 is gone; now on net POWERSC_-X1: J2.33, J2.34
- net POWERSC_-X_2 is gone; now on net POWERSC_-X2: J2.47, J2.48
- net SUP_12V0 is gone; now on net SUP_12V: J15.25, J15.26
- net SUP_3V3 is gone; now on net SUP_3V3_1: J23.5
- net Sunsensor -Y is gone; now on net Sunsensor_-Y: J2.45
- net Thruster-1 is gone; now on net Thruster_1: J10.25
- net Thruster-2 is gone; now on net Thruster_2: J10.26
- net Thurster_3 is gone; now on net Thruster_3: J10.35
- net SUP_5V_1: no longer J1.15
- net SUP_UNREG_1: now also J3.3 (C), J3.4 (D)
- net SUP_UNREG_3: no longer J3.3 (C), J3.4 (D)
- net MUX-CCB_UART (CCB_to_MainPIC) renamed MUX-CCB_UART (FPGA_to_MainPIC)
- net MUX-CCB_UART (MainPIC_to_CCB) renamed MUX-CCB_UART (MainPIC_to_FPGA)
- net OBC-MUX_UART (CCB/ThermalPIC_to_MainPIC) renamed OBC-MUX_UART (FPGA/ThermalPIC_to_MainPIC)
- net OBC-MUX_UART (MainPIC_to_CCB/ThermalPIC) renamed OBC-MUX_UART (MainPIC_to_FPGA/ThermalPIC)
- net POWERSC_-Z (nc): no longer names the net of J2.11
- net POWERSC_-Z (nc): no longer J2.12
- net UART (ADCS_to_CCB) renamed Earth_Sensor_UART (ADCS_to_RPi)
- net UART (CCB_to_ADCS) renamed Earth_Sensor_UART (RPi_to_ADCS)
- no-connect marks 75 -> 78
Other:
- company: (none) -> Kyutech
Changed lines of the file:
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@@
 	(title_block
 		(title "Turan-1_BPB")
-		(date "2026-03-17")
+		(date "2026-03-28")
+		(rev "v1")
+		(company "Kyutech")
+		(comment 1 "Turan-1 Backplane Board")
 	)
 	(text "DEP_SW4"
@@
 	)
 	(no_connect
+		(at 74.93 157.48)
+	)
+	(no_connect
 		(at 74.93 57.15)
 	)
@@
 	)
 	(no_connect
+		(at 52.07 49.53)
+	)
+	(no_connect
 		(at 163.83 190.5)
 	)
 	(no_connect
+		(at 52.07 157.48)
+	)
+	(no_connect
 		(at 52.07 41.91)
 	)
@@
 	(wire
 		(pts
-			(xy 74.93 157.48) (xy 77.47 157.48)
-		)
-		(stroke
-			(width 0)
-			(type default)
-		)
-	)
-	(wire
-		(pts
 			(xy 74.93 85.09) (xy 77.47 85.09)
 		)
@@
 	(wire
 		(pts
-			(xy 49.53 157.48) (xy 52.07 157.48)
-		)
-		(stroke
-			(width 0)
-			(type default)
-		)
-	)
-	(wire
-		(pts
 			(xy 365.76 147.32) (xy 368.3 147.32)
 		)
@@
 	(wire
 		(pts
-			(xy 49.53 49.53) (xy 52.07 49.53)
-		)
-		(stroke
-			(width 0)
-			(type default)
-		)
-	)
-	(wire
-		(pts
 			(xy 186.69 152.4) (xy 189.23 152.4)
 		)
@@
 		)
 	)
-	(global_label "Thurster_3"
+	(global_label "Thruster_3"
 		(shape input)
 		(at 167.64 76.2 180)
@@
 		)
 	)
-	(global_label "SUP_12V0"
+	(global_label "SUP_12V"
 		(shape input)
 		(at 285.75 201.93 180)
@@
 		)
 		(property "Intersheetrefs" "${INTERSHEET_REFS}"
-			(at 273.2701 201.93 0)
+			(at 274.4796 201.93 0)
 			(effects
 				(font
@@
 		)
 	)
-	(global_label "SUP_5V_1"
-		(shape input)
-		(at 49.53 49.53 180)
-		(fields_autoplaced yes)
-		(effects
-			(font
-				(size 1.27 1.27)
-			)
-			(justify right)
-		)
-		(property "Intersheetrefs" "${INTERSHEET_REFS}"
-			(at 37.292 49.53 0)
-			(effects
-				(font
-					(size 1.27 1.27)
-				)
-				(justify right)
-				(hide yes)
-			)
-		)
-	)
-	(global_label "POWERSC_-X_1"
+	(global_label "POWERSC_-X1"
 		(shape input)
 		(at 77.47 185.42 0)
@@
 		)
 		(property "Intersheetrefs" "${INTERSHEET_REFS}"
-			(at -81.42 -23.98 0)
+			(at 94.3646 185.42 0)
 			(effects
 				(font
@@
 		)
 	)
-	(global_label "OBC-CCB DIO ON{slash}OFF (MainPIC_to_CCB)"
+	(global_label "OBC-CCB_DIO_ON{slash}OFF (MainPIC_to_CCB)"
 		(shape input)
 		(at 285.75 138.43 180)
@@
 		)
 	)
-	(global_label "UART (CCB_to_ADCS)"
+	(global_label "Earth_Sensor_UART (RPi_to_ADCS)"
 		(shape input)
 		(at 285.75 146.05 180)
@@
 		)
 		(property "Intersheetrefs" "${INTERSHEET_REFS}"
-			(at 262.9891 146.05 0)
+			(at 250.3498 146.05 0)
 			(effects
 				(font
@@
 		)
 	)
-	(global_label "Thruster-2"
+	(global_label "Thruster_2"
 		(shape input)
 		(at 193.04 63.5 0)
@@
 		)
 		(property "Intersheetrefs" "${INTERSHEET_REFS}"
-			(at 206.4875 63.5 0)
+			(at 205.8827 63.5 0)
 			(effects
 				(font
@@
 		)
 	)
-	(global_label "OBC-MUX_UART (MainPIC_to_CCB{slash}ThermalPIC)"
+	(global_label "OBC-MUX_UART (MainPIC_to_FPGA{slash}ThermalPIC)"
 		(shape input)
 		(at 300.99 66.04 180)
@@
 		)
 		(property "Intersheetrefs" "${INTERSHEET_REFS}"
-			(at 253.1921 66.04 0)
+			(at 252.2849 66.04 0)
 			(effects
 				(font
@@
 		)
 	)
-	(global_label "SUP_UNREG_3"
+	(global_label "SUP_UNREG_1"
 		(shape input)
 		(at 50.8 134.62 180)
@@
 		)
 	)
-	(global_label "SUP_12V0"
+	(global_label "SUP_12V"
 		(shape input)
 		(at 285.75 199.39 180)
@@
 		)
 		(property "Intersheetrefs" "${INTERSHEET_REFS}"
-			(at 273.2701 199.39 0)
+			(at 274.4796 199.39 0)
 			(effects
 				(font
@@
 		)
 	)
-	(global_label "MUX-CCB_UART (CCB_to_MainPIC)"
+	(global_label "MUX-CCB_UART (FPGA_to_MainPIC)"
 		(shape input)
 		(at 285.75 143.51 180)
@@
 		)
 		(property "Intersheetrefs" "${INTERSHEET_REFS}"
-			(at 249.9868 143.51 0)
+			(at 249.0796 143.51 0)
 			(effects
 				(font
@@
 		)
 	)
-	(global_label "UART (ADCS_to_CCB)"
+	(global_label "Earth_Sensor_UART (ADCS_to_RPi)"
 		(shape input)
 		(at 285.75 148.59 180)
@@
 		)
 		(property "Intersheetrefs" "${INTERSHEET_REFS}"
-			(at 262.9891 148.59 0)
+			(at 250.3498 148.59 0)
 			(effects
 				(font
@@
 		)
 	)
-	(global_label "UART (CCB_to_ADCS)"
+	(global_label "Earth_Sensor_UART (RPi_to_ADCS)"
 		(shape input)
 		(at 161.29 154.94 180)
@@
 		)
 		(property "Intersheetrefs" "${INTERSHEET_REFS}"
-			(at 138.5291 154.94 0)
+			(at 125.8898 154.94 0)
 			(effects
 				(font
@@
 		)
 	)
-	(global_label "UART (ADCS_to_CCB)"
+	(global_label "Earth_Sensor_UART (ADCS_to_RPi)"
 		(shape input)
 		(at 189.23 154.94 0)
@@
 		)
 		(property "Intersheetrefs" "${INTERSHEET_REFS}"
-			(at 211.9909 154.94 0)
+			(at 224.6302 154.94 0)
 			(effects
 				(font
@@
 		)
 	)
-	(global_label "MUX-CCB_UART (MainPIC_to_CCB)"
+	(global_label "MUX-CCB_UART (MainPIC_to_FPGA)"
 		(shape input)
 		(at 285.75 140.97 180)
@@
 		)
 		(property "Intersheetrefs" "${INTERSHEET_REFS}"
-			(at 249.9868 140.97 0)
+			(at 249.0796 140.97 0)
 			(effects
 				(font
@@
 		)
 	)
-	(global_label "Sunsensor -Y"
+	(global_label "Sunsensor_-Y"
 		(shape input)
 		(at 49.53 200.66 180)
@@
 		)
 		(property "Intersheetrefs" "${INTERSHEET_REFS}"
-			(at -94.12 -23.94 0)
+			(at 33.1797 200.66 0)
 			(effects
 				(font
@@
 		)
 	)
-	(global_label "OBC-MUX_UART (CCB{slash}ThermalPIC_to_MainPIC)"
+	(global_label "OBC-MUX_UART (FPGA{slash}ThermalPIC_to_MainPIC)"
 		(shape input)
 		(at 328.93 66.04 0)
@@
 		)
 		(property "Intersheetrefs" "${INTERSHEET_REFS}"
-			(at 376.7279 66.04 0)
+			(at 377.6351 66.04 0)
 			(effects
 				(font
@@
 		)
 	)
-	(global_label "POWERSC_-Z (nc)"
-		(shape input)
-		(at 77.47 157.48 0)
-		(fields_autoplaced yes)
-		(effects
-			(font
-				(size 1.27 1.27)
-			)
-			(justify left)
-		)
-		(property "Intersheetrefs" "${INTERSHEET_REFS}"
-			(at -81.42 -23.92 0)
-			(effects
-				(font
-					(size 1.27 1.27)
-				)
-				(justify left)
-				(hide yes)
-			)
-		)
-	)
 	(global_label "SPI_CS (ADCS_to_FM2)"
 		(shape input)
@@
 		)
 	)
-	(global_label "POWERSC_-X_2"
+	(global_label "POWERSC_-X2"
 		(shape input)
 		(at 77.47 203.2 0)
@@
 		)
 		(property "Intersheetrefs" "${INTERSHEET_REFS}"
-			(at -81.42 -24 0)
+			(at 94.3646 203.2 0)
 			(effects
 				(font
@@
 		)
 	)
-	(global_label "Thruster-1"
+	(global_label "Thruster_1"
 		(shape input)
 		(at 167.64 63.5 180)
@@
 		)
 		(property "Intersheetrefs" "${INTERSHEET_REFS}"
-			(at 154.1925 63.5 0)
+			(at 154.7973 63.5 0)
 			(effects
 				(font
@@
 		)
 	)
-	(global_label "POWERSC_-X_2"
+	(global_label "POWERSC_-X2"
 		(shape input)
 		(at 49.53 203.2 180)
@@
 		)
 		(property "Intersheetrefs" "${INTERSHEET_REFS}"
-			(at -94.12 -24 0)
+			(at 32.6354 203.2 0)
 			(effects
 				(font
@@
 		)
 	)
-	(global_label "SUP_UNREG_3"
+	(global_label "SUP_UNREG_1"
 		(shape input)
 		(at 76.2 134.62 0)
@@
 		)
 	)
-	(global_label "POWERSC_-Z (nc)"
-		(shape input)
-		(at 49.53 157.48 180)
-		(fields_autoplaced yes)
-		(effects
-			(font
-				(size 1.27 1.27)
-			)
-			(justify right)
-		)
-		(property "Intersheetrefs" "${INTERSHEET_REFS}"
-			(at -94.12 -23.92 0)
-			(effects
-				(font
-					(size 1.27 1.27)
-				)
-				(justify right)
-				(hide yes)
-			)
-		)
-	)
-	(global_label "SUP_3V3"
+	(global_label "SUP_3V3_1"
 		(shape input)
 		(at 365.76 149.86 180)
@@
 		)
 		(property "Intersheetrefs" "${INTERSHEET_REFS}"
-			(at 354.4896 149.86 0)
+			(at 352.3125 149.86 0)
 			(effects
 				(font
@@
 		)
 	)
-	(global_label "POWERSC_-X_1"
+	(global_label "POWERSC_-X1"
 		(shape input)
 		(at 49.53 185.42 180)
@@
 		)
 		(property "Intersheetrefs" "${INTERSHEET_REFS}"
-			(at -94.12 -23.98 0)
+			(at 32.6354 185.42 0)
 			(effects
 				(font

Commit message: Microelectronic components placed onto the back of BPB
Parts:
- removed J1, J10, J2: A3C-50DA-2DSA_71_, Custom-Footprints:Hirose_A3C-50DA-2DSC(71), symbol Custom-Symbols:A3C-50DA-2DSA_71_
- removed J9: A3C-50DA-2DSA_71_, Custom-Footprints:Hirose_A3C-50DA-2DSC(71)_Mirrored, symbol Custom-Symbols:A3C-50DA-2DSA_71_
- added J1, J2, J5, J6: A3C-50DA-2DSA_71_, Custom-Footprints:Hirose_A3C-50DA-2DSC(71)_Mirrored, symbol Custom-Symbols:A3C-50DA-2DSA_71_Mirrored
- J16: footprint Custom-Footprints:Hirose_A3C-50DA-2DSC(71)_Mirrored -> Custom-Footprints:Hirose_A3C-50DA-2DSC(71)
- J17, J18: footprint Custom-Footprints:Hirose_A3C-4DA-2DSA(71)_Mirrored -> Custom-Footprints:Hirose_A3C-4DA-2DSA(71)
- J3, J4: footprint Custom-Footprints:Hirose_A3C-4DA-2DSA(71) -> Custom-Footprints:Hirose_A3C-4DA-2DSA(71)_Mirrored
Connections:
- net ADB-ThermalPIC_PWR_ON_DIO: now also J5.33
- net ADB-ThermalPIC_UART (Debug_to_Thermal): now also J5.27
- net ADCS-ADB UART (ADCSPIC_to_Debug): now also J5.19, J6.20
- net ADCS-ADB UART (ADCSSTM32_to_Debug): now also J5.45, J6.48
- net ADCS-ADB UART (Debug_to_ADCSPIC): now also J5.20, J6.19
- net ADCS-ADB UART (Debug_to_ADCSSTM32): now also J5.44, J6.47
- net ADCS_STM32_SWCLK: now also J5.32, J6.41
- net ADCS_STM32_SWDIO: now also J5.43, J6.42
- net ANALOG_RSSI (UHF_to_RelayPIC): now also J1.48, J5.34
- net ANALOG_TEMP (UHF_to_RelayPIC): now also J1.47, J5.39
- net Battery_Voltage_Check: now also J2.22, J5.22
- net Charging: now also J2.37, J2.38, J5.37, J5.38
- net DEP_SW12: now also J2.40, J2.41
- net DEP_SW3: now also J2.42
- net DEP_SW4: now also J2.43
- net DIO_1 (ComPIC_to_GMSK_EN): now also J1.44
- net DIO_2 (ComPIC_to_CW_EN): now also J1.45
- net DIO_3 (ComPIC_to_UHF CW_KEY): now also J1.46
- net DIO_Fault_Indicator: now also J5.16
- net DIO_HW_Reset: now also J5.10
- net DIO_Thruster_Active: now also J5.15
- net DIO_UHF_Antenna_Deploy: now also J2.21, J5.42
- net E-MGM_3v3: now also J6.22
- net E-MGM_SCL: now also J6.38
- net E-MGM_SDA: now also J6.37
- net Earth_Sensor_UART (ADCS_to_RPi): now also J6.18
- net Earth_Sensor_UART (RPi_to_ADCS): now also J6.17
- net GND_BAT: now also J22.2, J2.17
- net GND_SYS: now also J1.13, J1.14, J2.13, J2.14, J5.13, J5.14, J6.13, J6.14; no longer J22.2
- net GPS_1PPS: now also J6.44
- net GPS_3v3: now also J6.43
- net Kill_SW (MainPIC_to_EPS): now also J2.39
- net MCLR_ADCS_PIC: now also J5.7, J6.5
- net MCLR_ComPIC: now also J5.5
- net MCLR_EpsPIC: now also J2.3, J5.3
- net MCLR_MainPIC: now also J5.6
- net MCLR_ResetPIC: now also J5.4
- net MCLR_StartPIC: now also J5.8
- net MCLR_ThermalPIC: now also J5.9
- net MUX-ADB UART_1 (MainPIC_to_RelayPIC): now also J5.11
- net MUX-ADB UART_1 (RelayPIC_to_MainPIC): now also J5.12
- net MUX-ADCS UART (ADCS_to_MainPIC): now also J6.4
- net MUX-ADCS UART (MainPIC_to_ADCS): now also J6.3
- net MUX-EPS1 UART (EPS1PIC_to_MainPIC): now also J2.20
- net MUX-EPS1 UART (MainPIC_to_EPS1PIC): now also J2.19
- net OBC-ADB DIO ON/OFF (MainPIC_to_RelayPIC): now also J5.41
- net OBC-ADB UART_2 (Debug_to_MainPIC): now also J5.18
- net OBC-ADB UART_2 (MainPIC_to_Debug): now also J5.17
- net OBC-ADB UART_3 (RelayPIC_to_ComPIC): now also J5.21
- net OBC-ADCS_DIO_ON/OFF (MainPIC_to_ADCS): now also J6.46
- net PGC: now also J2.1, J5.1, J6.1
- net PGD: now also J2.2, J5.2, J6.2
- net POWERSC_+X: now also J2.27, J2.28
- net POWERSC_+Y: now also J2.7, J2.8
- net POWERSC_-X1: now also J2.33, J2.34
- net POWERSC_-X2: now also J2.47, J2.48
- net RAW_POWER: now also J2.29, J2.30
- net S-band_RX_Analog_AGC_RSSI: now also J5.47
- net S-band_RX_Analog_Freq_ERR: now also J5.46
- net S-band_RX_NRZ_1K_CLK: now also J5.31
- net S-band_RX_NRZ_1K_DATA: now also J5.40
- net S-band_RX_NRZ_4K_CLK: now also J5.30
- net S-band_RX_NRZ_4K_DATA: now also J5.29
- net S-band_TX_Analog_Temperature: now also J5.48
- net SPI _MOSI (ADCS_to_FM2): now also J6.30
- net SPI_CS (ADCS_to_FM2): now also J6.29
- net SPI_MISO (FM2_to_ADCS): now also J6.27
- net SPI_SCK (ADCS_to_FM2): now also J6.28
- net SUP_3V3_1: now also J1.49, J1.50, J2.49, J2.50, J5.49, J5.50
- net SUP_5V_1: now also J2.15, J2.16
- net SUP_5V_2: now also J2.25, J2.26
- net SUP_UNREG_1: now also J1.23, J1.24, J2.23, J2.24, J5.23, J5.24
- net SUP_UNREG_2: now also J2.35, J2.36
- net SUP_UNREG_3: now also J6.35, J6.36
- net Sunsensor_+X: now also J6.7
- net Sunsensor_+Y: now also J6.9
- net Sunsensor_+Z: now also J6.11
- net Sunsensor_-X: now also J6.8
- net Sunsensor_-Y: now also J2.45, J6.10
- net Sunsensor_-Z1: now also J6.12
- net Sunsensor_-Z2: now also J6.21
- net TEMP_+X: now also J2.31
- net TEMP_+Y: now also J2.10
- net TEMP_+Z: now also J2.46
- net TEMP_-X: now also J2.32
- net TEMP_-Z: now also J2.9
- net TEMP_BPB: now also J2.44
- net ThermalPIC-ADB_UART (Thermal_to_Debug): now also J5.28
- net Thruster_1: now also J5.25
- net Thruster_2: now also J5.26
- net Thruster_3: now also J5.35
- net UART (ADCS_to_GPS): now also J6.31
- net UART (ComPIC_to_UHF): now also J1.8
- net UART (GPS_to_ADCS): now also J6.32
- net UART (UHF_to_ComPIC): now also J1.7
- no-connect marks 78 -> 86
Other:
- moved on the sheet: J15, J16, J23, J3, J4
