File: BP-PCB-ICs.kicad_sch (KiCad schematic)
At the start: 50 parts, among them IC1 LMT84DCKT, Q1 SSM6K514NU,LF, Q2 SSM6K514NU,LF, Q3 SSM6K514NU,LF, Q4 SSM6K514NU,LF, Q5 SSM6K514NU,LF, Q6 SSM6K514NU,LF, U1 LTC4361CTS8-2TRMPBF, U2 LTC4361CTS8-2TRMPBF, U6 LTC4389IMS-4#PBF, U7 LTC4389IMS-4#PBF

Commit message: Finished routing and NO DRC errors
Parts:
- removed R18: 5 Ohm, Resistor_SMD:R_0805_2012Metric, symbol Device:R_US
- removed U7: LTC4389IMS-4#PBF, Custom-Footprints:LTC4380IMS-4#PBF, symbol Custom-Symbols:LTC4380IMS-4#PBF
- added U4: LTC4380IMS-4#PBF, Custom-Footprints:LTC4380IMS-4#PBF, symbol Custom-Symbols:LTC4380IMS-4#PBF
- C1, C2: LCSC Part (none) -> C1712
- C10, C15: LCSC Part (none) -> C1745
- C12, C16: LCSC Part (none) -> C45783
- C13, C5, C6, C8: LCSC Part (none) -> C1746
- C14, C9: LCSC Part (none) -> C1770
- C17: LCSC Part (none) -> C29926
- C3, C4: LCSC Part (none) -> C77062
- D1: LCSC Part (none) -> C151430
- IC1: LCSC Part (none) -> C2860524
- Q1, Q2, Q3, Q4, Q5, Q6: LCSC Part (none) -> C6235373
- R1: LCSC Part (none) -> C702831
- R10, R9: LCSC Part (none) -> C858607
- R11, R13, R4, R6: LCSC Part (none) -> C702829
- R12, R5: LCSC Part (none) -> C17470
- R14, R7: LCSC Part (none) -> C49330262
- R15, R8: LCSC Part (none) -> C702857
- R16, R17: value 25m Ohm -> 25m; LCSC Part (none) -> C858607
- R19, R21: LCSC Part (none) -> C2828711
- R2: value 5 Ohm -> 2.5 Ohm; LCSC Part (none) -> C409739
- R20, R3: LCSC Part (none) -> C409739
- R23: LCSC Part (none) -> C702869
- U1, U2: LCSC Part (none) -> C688257
- U6: value LTC4389IMS-4#PBF -> LTC4380IMS-4#PBF; LCSC Part (none) -> C688474
Connections:
- net  V_IN (Unreg2 OCP to S-band RX): now also U6.5 (OUT)
- net  V_IN (Unreg2 OCP to S-band TX): now also U4.5 (OUT); no longer U6.5 (OUT)
- net DIO_S-Band_RX_ON/OFF: now also U6.9 (ON)
- net DIO_S-Band_TX_ON/OFF: now also U4.9 (ON); no longer U6.9 (ON)
- net GND_SYS: now also U4.6 (SEL), U4.8 (GND)
- net at C8.1, R4.2: now also U4.2 (VCC); no longer U6.2 (VCC)
- net at R14.1, R15.1: now also U6.3 (GATE)
- net at Q3.1 (D_1), Q3.2 (D_2), Q3.5 (D_3)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: now also U4.4 (SNS); no longer U6.4 (SNS)
- net at U6.1 (DRN): now also R12.2; no longer R5.2
- net at U6.10 (TMR): now also C14.1; no longer C9.1
- net at R7.1, R8.1: now also U4.3 (GATE); no longer U6.3 (GATE)
- net at C13.1, R11.2: now also U6.2 (VCC)
- net at Q5.1 (D_1), Q5.2 (D_2), Q5.5 (D_3)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: now also U6.4 (SNS)
- new net: R5.2, U4.1 (DRN)
- new net: C9.1, U4.10 (TMR)

Commit message: ERC errors eleminated from schematic
Parts:
- U1, U2: LCSC Part C688257 -> (none)

Commit message: Corrected OCP values in schematic and fixed PCB layout
Parts:
- removed R10, R17: 25m, Resistor_SMD:R_0805_2012Metric, symbol Device:R_Small_US
- removed U4, U6: LTC4380IMS-4#PBF, Custom-Footprints:LTC4380IMS-4#PBF, symbol Custom-Symbols:LTC4380IMS-4#PBF
- added U4, U6: LTC4380IMS-2#PBF, Custom-Footprints:LTC4380IMS-2#PBF, symbol Custom-Symbols:LTC4380IMS-2#PBF
Connections:
- net  V_IN (Unreg2 OCP to S-band RX): now also U6.5 (OUT)
- net  V_IN (Unreg2 OCP to S-band TX): now also U4.5 (OUT)
- net DIO_S-Band_RX_ON/OFF: now also U6.9 (ON)
- net DIO_S-Band_TX_ON/OFF: now also U4.9 (ON)
- net GND_SYS: now also U4.6 (SEL), U4.8 (GND), U6.6 (SEL), U6.8 (GND)
- net at C8.1, R4.2: now also U4.2 (VCC)
- net at R14.1, R15.1: now also U6.3 (GATE)
- net at Q3.1 (D_1), Q3.2 (D_2), Q3.5 (D_3)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: now also U4.4 (SNS)
- net at C13.1, R11.2: now also U6.2 (VCC)
- net at Q5.1 (D_1), Q5.2 (D_2), Q5.5 (D_3)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: now also U6.4 (SNS)
- net at C14.1: now also U6.10 (TMR)
- net at R7.1, R8.1: now also U4.3 (GATE)
- net at R12.2: now also U6.1 (DRN)
- net at R5.2: now also U4.1 (DRN)
- net at C9.1: now also U4.10 (TMR)

Commit message: BBM version requested for fabrication
Parts:
- removed U1, U2: LTC4361CTS8-2TRMPBF, Custom-Footprints:LTC4361HTS8, symbol Custom-Symbols:LTC4361CTS8-2TRMPBF
- added U1, U2: LTC4361-2, Custom-Footprints:LTC4361HTS8, symbol Custom-Symbols:LTC4361-2
- U4, U6: LCSC Part C117125 -> C688471
Connections:
- net GND_SYS: now also U1.1 (~{ON}), U1.4 (GND), U2.1 (~{ON}), U2.4 (GND)
- net SUP_3V3_1: now also U1.5 (IN), U2.5 (IN)
- net TEMP_3v3_MX: now also U1.2 (OUT)
- net TEMP_3v3_PX: now also U2.2 (OUT)
- net at Q1.1 (D_1), Q1.2 (D_2), Q1.5 (D_3)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: now also U1.6 (SENSE)
- net at C3.1, Q1.3 (G): now also U1.7 (GATE)
- net at Q2.1 (D_1), Q2.2 (D_2), Q2.5 (D_3)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: now also U2.6 (SENSE)
- net at C4.1, Q2.3 (G): now also U2.7 (GATE)
Changed lines of the file:
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@@
 	)
 	(symbol
+		(lib_id "Custom-Symbols:LTC4361-2")
+		(at 327.66 50.8 0)
+		(unit 1)
+		(exclude_from_sim no)
+		(in_bom yes)
+		(on_board yes)
+		(dnp no)
+		(fields_autoplaced yes)
+		(property "Reference" "U2"
+			(at 327.66 33.02 0)
+			(effects
+				(font
+					(size 2.0848 1.772)
+				)
+			)
+		)
+		(property "Value" "LTC4361-2"
+			(at 327.66 36.83 0)
+			(effects
+				(font
+					(size 2.0859 1.773)
+				)
+			)
+		)
+		(property "Footprint" "Custom-Footprints:LTC4361HTS8"
+			(at 330.2 35.052 0)
+			(effects
+				(font
+					(size 1.27 1.27)
+				)
+				(hide yes)
+			)
+		)
+		(property "Datasheet" ""
+			(at 327.66 50.8 0)
+			(effects
+				(font
+					(size 1.27 1.27)
+				)
+				(hide yes)
+			)
+		)
+		(property "Description" ""
+			(at 327.66 50.8 0)
+			(effects
+				(font
+					(size 1.27 1.27)
+				)
+				(hide yes)
+			)
+		)
+		(property "LCSC Part" "C688273"
+			(at 327.66 50.8 0)
+			(effects
+				(font
+					(size 1.27 1.27)
+				)
+				(hide yes)
+			)
+		)
+		(pin "4"
+		)
+		(pin "6"
+		)
+		(pin "1"
+		)
+		(pin "5"
+		)
+		(pin "3"
+		)
+		(pin "7"
+		)
+		(pin "8"
+		)
+		(pin "2"
+		)
+		(instances
+			(project ""
+				(path "/da3a05e5-7f1e-43cd-9425-16ff965529d1/b13c3f99-87b6-43ee-99ee-c97ccd64f2f6"
+					(reference "U2")
+					(unit 1)
+				)
+			)
+		)
+	)
+	(symbol
 		(lib_id "Device:R_Small_US")
 		(at 102.87 81.28 0)
@@
 			)
 		)
-		(property "LCSC Part" "C117125"
+		(property "LCSC Part" "C688471 "
 			(at 54.61 66.04 0)
 			(effects
@@
 	)
 	(symbol
-		(lib_id "Custom-Symbols:LTC4361CTS8-2TRMPBF")
-		(at 327.66 50.8 0)
-		(unit 1)
-		(exclude_from_sim no)
-		(in_bom yes)
-		(on_board yes)
-		(dnp no)
-		(fields_autoplaced yes)
-		(property "Reference" "U2"
-			(at 327.66 33.02 0)
-			(effects
-				(font
-					(size 2.0848 1.772)
-				)
-			)
-		)
-		(property "Value" "LTC4361CTS8-2TRMPBF"
-			(at 327.66 36.83 0)
-			(effects
-				(font
-					(size 2.0859 1.773)
-				)
-			)
-		)
-		(property "Footprint" "Custom-Footprints:LTC4361HTS8"
-			(at 312.42 29.21 0)
-			(effects
-				(font
-					(size 1.27 1.27)
-				)
-				(hide yes)
-			)
-		)
-		(property "Datasheet" ""
-			(at 327.66 50.8 0)
-			(effects
-				(font
-					(size 1.27 1.27)
-				)
-				(hide yes)
-			)
-		)
-		(property "Description" ""
-			(at 327.66 50.8 0)
-			(effects
-				(font
-					(size 1.27 1.27)
-				)
-				(hide yes)
-			)
-		)
-		(pin "5"
-		)
-		(pin "7"
-		)
-		(pin "8"
-		)
-		(pin "2"
-		)
-		(pin "3"
-		)
-		(pin "6"
-		)
-		(pin "4"
-		)
-		(pin "1"
-		)
-		(instances
-			(project ""
-				(path "/da3a05e5-7f1e-43cd-9425-16ff965529d1/b13c3f99-87b6-43ee-99ee-c97ccd64f2f6"
-					(reference "U2")
-					(unit 1)
-				)
-			)
-		)
-	)
-	(symbol
 		(lib_id "Custom-Symbols:LTC4380IMS-2#PBF")
 		(at 54.61 180.34 0)
@@
 			)
 		)
-		(property "LCSC Part" "C117125"
+		(property "LCSC Part" "C688471 "
 			(at 54.61 180.34 0)
 			(effects
@@
 	)
 	(symbol
-		(lib_name "LTC4361CTS8-2TRMPBF_1")
-		(lib_id "Custom-Symbols:LTC4361CTS8-2TRMPBF")
+		(lib_id "Custom-Symbols:LTC4361-2")
 		(at 330.2 144.78 0)
 		(unit 1)
@@
 			)
 		)
-		(property "Value" "LTC4361CTS8-2TRMPBF"
+		(property "Value" "LTC4361-2"
 			(at 330.2 130.81 0)
 			(effects
@@
 		)
 		(property "Footprint" "Custom-Footprints:LTC4361HTS8"
-			(at 314.96 123.19 0)
+			(at 332.74 129.032 0)
 			(effects
 				(font
@@
 			)
 		)
-		(pin "7"
+		(property "LCSC Part" "C688273"
+			(at 330.2 144.78 0)
+			(effects
+				(font
+					(size 1.27 1.27)
+				)
+				(hide yes)
+			)
+		)
+		(pin "5"
 		)
 		(pin "8"
@@
 		(pin "3"
 		)
-		(pin "5"
+		(pin "7"
 		)
 		(pin "1"
@@
 		(pin "4"
 		)
-		(pin "2"
-		)
 		(pin "6"
 		)
+		(pin "2"
+		)
 		(instances
